Commit message: feat: Menagerie-style MJCF models and drive-based joint parameters
- MJCF restructured (robot-only files, per-robot scenes, home keyframe)
- Joint limits, armature and friction from drive configs and datasheets
- URDF, Isaac Lab config, package.xml and docs cleanup; new MuJoCo tests

File: urdf/common/_gazebo.xacro (robot description, xacro)
@@ -1,6 +1,9 @@
 <?xml version="1.0"?>
 <robot xmlns:xacro="http://www.ros.org/wiki/xacro">
-  <!-- Resolved at include time relative to this file; no $(find), works from source and install -->
-  <xacro:property name="config_dir" value="${xacro.abs_filename('../../config')}" lazy_eval="false" />
+  <!-- Resolved at include time relative to this file; no $(find), works from source and install.
+       abs_filename() is relative when xacro gets a relative path, so prefix the working directory then. -->
+  <xacro:property name="config_rel" value="${xacro.abs_filename('../../config')}" lazy_eval="false" />
+  <xacro:property name="config_dir" value="${config_rel if config_rel.startswith('/') else '$(cwd)/' + config_rel}"
+    lazy_eval="false" />
   <!-- imu_xyz: MJCF imu site pos -->
   <xacro:macro name="gazebo_block" params="robot imu_xyz">

File: urdf/common/_materials.xacro (robot description, xacro)
@@ -13,6 +13,3 @@
     <color rgba="1 0.41 0 1" />
   </material>
-  <material name="invisible">
-    <color rgba="0 0 0 0.001" />
-  </material>
 </robot>

File: urdf/hb40/_hb40_leg_macro.xacro (robot description, xacro)
@@ -47,5 +47,4 @@
           <cylinder length="0.11" radius="0.05" />
         </geometry>
-        <material name="invisible" />
       </collision>
     </link>
@@ -68,5 +67,4 @@
           <cylinder length="0.0625" radius="0.01" />
         </geometry>
-        <material name="invisible" />
       </collision>
       <collision>
@@ -75,13 +73,8 @@
           <cylinder length="0.2" radius="0.015" />
         </geometry>
-        <material name="invisible" />
       </collision>
     </link>
     <!-- Foot : massless -->
     <link name="${prefix}_foot">
-      <inertial>
-        <mass value="0" />
-        <inertia ixx="0" ixy="0" ixz="0" iyy="0" iyz="0" izz="0" />
-      </inertial>
       <visual>
         <geometry>
@@ -92,5 +85,5 @@
       <collision>
         <geometry>
-          <sphere radius="0.02" />
+          <sphere radius="0.021" />
         </geometry>
       </collision>
@@ -102,6 +95,6 @@
       <origin xyz="${j0_xyz}" rpy="${j0_rpy}" />
       <axis xyz="1 0 0" />
-      <limit effort="27.0" lower="-1.570796" upper="1.570796" velocity="25.0" />
-      <dynamics damping="0.1" friction="0.48" />
+      <limit effort="15.0" lower="-1.570796" upper="1.570796" velocity="59.0" />
+      <dynamics damping="0.1" friction="0.51" />
     </joint>
     <joint name="${prefix}_j1" type="revolute">
@@ -110,6 +103,6 @@
       <origin xyz="${j1_xyz}" rpy="${j1_rpy}" />
       <axis xyz="1 0 0" />
-      <limit effort="27.0" lower="-1.570796" upper="1.570796" velocity="25.0" />
-      <dynamics damping="0.1" friction="0.48" />
+      <limit effort="15.0" lower="-1.570796" upper="1.570796" velocity="59.0" />
+      <dynamics damping="0.1" friction="0.51" />
     </joint>
     <joint name="${prefix}_j2" type="revolute">
@@ -118,6 +111,6 @@
       <origin xyz="${j2_xyz}" rpy="${j2_rpy}" />
       <axis xyz="1 0 0" />
-      <limit effort="27.0" lower="${j2_lower}" upper="${j2_upper}" velocity="25.0" />
-      <dynamics damping="0.1" friction="0.48" />
+      <limit effort="15.0" lower="${j2_lower}" upper="${j2_upper}" velocity="59.0" />
+      <dynamics damping="0.1" friction="0.51" />
     </joint>
     <joint name="${prefix}_jFoot" type="fixed">

File: urdf/hb40/hb40.urdf (robot description, URDF)
Before this commit: robot hb40, 17 links, 16 joints
Links:
- link fl_foot: mass 0 -> None; geometry collision sphere radius=0.021; visual sphere radius=0.021
- link fr_foot: mass 0 -> None; geometry collision sphere radius=0.021; visual sphere radius=0.021
- link rl_foot: mass 0 -> None; geometry collision sphere radius=0.021; visual sphere radius=0.021
- link rr_foot: mass 0 -> None; geometry collision sphere radius=0.021; visual sphere radius=0.021
Joints:
- joint fl_j0: limit lower=-1.570796 upper=1.570796 effort=27.0 velocity=25.0 -> lower=-1.570796 upper=1.570796 effort=15.0 velocity=59.0
- joint fl_j1: limit lower=-1.570796 upper=1.570796 effort=27.0 velocity=25.0 -> lower=-1.570796 upper=1.570796 effort=15.0 velocity=59.0
- joint fl_j2: limit lower=0 upper=2.53 effort=27.0 velocity=25.0 -> lower=0 upper=2.53 effort=15.0 velocity=59.0
- joint fr_j0: limit lower=-1.570796 upper=1.570796 effort=27.0 velocity=25.0 -> lower=-1.570796 upper=1.570796 effort=15.0 velocity=59.0
- joint fr_j1: limit lower=-1.570796 upper=1.570796 effort=27.0 velocity=25.0 -> lower=-1.570796 upper=1.570796 effort=15.0 velocity=59.0
- joint fr_j2: limit lower=-2.53 upper=0 effort=27.0 velocity=25.0 -> lower=-2.53 upper=0 effort=15.0 velocity=59.0
- joint rl_j0: limit lower=-1.570796 upper=1.570796 effort=27.0 velocity=25.0 -> lower=-1.570796 upper=1.570796 effort=15.0 velocity=59.0
- joint rl_j1: limit lower=-1.570796 upper=1.570796 effort=27.0 velocity=25.0 -> lower=-1.570796 upper=1.570796 effort=15.0 velocity=59.0
- joint rl_j2: limit lower=0 upper=2.53 effort=27.0 velocity=25.0 -> lower=0 upper=2.53 effort=15.0 velocity=59.0
- joint rr_j0: limit lower=-1.570796 upper=1.570796 effort=27.0 velocity=25.0 -> lower=-1.570796 upper=1.570796 effort=15.0 velocity=59.0
- joint rr_j1: limit lower=-1.570796 upper=1.570796 effort=27.0 velocity=25.0 -> lower=-1.570796 upper=1.570796 effort=15.0 velocity=59.0
- joint rr_j2: limit lower=-2.53 upper=0 effort=27.0 velocity=25.0 -> lower=-2.53 upper=0 effort=15.0 velocity=59.0

File: urdf/hb40/hb40.urdf.xacro (robot description, xacro)
@@ -3,4 +3,7 @@
   <!-- sim: none | mock | gazebo -->
   <xacro:arg name="sim" default="none" />
+  <xacro:if value="${'$(arg sim)' not in ['none', 'mock', 'gazebo']}">
+    ${xacro.fatal("sim must be none, mock or gazebo, got '$(arg sim)'")}
+  </xacro:if>
   <xacro:include filename="../common/_materials.xacro" />
   <xacro:include filename="_hb40_leg_macro.xacro" />
@@ -21,5 +24,4 @@
         <box size="0.27 0.178 0.1" />
       </geometry>
-      <material name="invisible" />
     </collision>
   </link>

File: urdf/hb50/_hb50_leg_macro.xacro (robot description, xacro)
@@ -9,5 +9,5 @@
       l0_inertial_xyz l0_visual_rpy:='0 0 0'
       j1_xyz j1_rpy j1_lower j1_upper
-      l1_inertial_xyz l1_ixx l1_iyy l1_izz l1_visual_rpy l1_mesh
+      l1_mass l1_inertial_xyz l1_ixx l1_iyy l1_izz l1_visual_rpy l1_mesh
       l1_collision2_xyz l1_collision2_rpy
       j2_xyz j2_rpy j2_lower j2_upper
@@ -36,5 +36,5 @@
       <inertial>
         <origin xyz="${l1_inertial_xyz}" />
-        <mass value="1.784" />
+        <mass value="${l1_mass}" />
         <inertia ixx="${l1_ixx}" ixy="0" ixz="0" iyy="${l1_iyy}" iyz="0" izz="${l1_izz}" />
       </inertial>
@@ -51,5 +51,4 @@
           <cylinder length="0.132" radius="0.051" />
         </geometry>
-        <material name="invisible" />
       </collision>
       <collision>
@@ -58,5 +57,4 @@
           <box size="0.028 0.22 0.052" />
         </geometry>
-        <material name="invisible" />
       </collision>
     </link>
@@ -80,5 +78,4 @@
           <cylinder length="0.06" radius="0.012" />
         </geometry>
-        <material name="invisible" />
       </collision>
       <collision>
@@ -87,13 +84,8 @@
           <cylinder length="0.196" radius="0.016" />
         </geometry>
-        <material name="invisible" />
       </collision>
     </link>
     <!-- Foot : massless -->
     <link name="${prefix}_foot">
-      <inertial>
-        <mass value="0" />
-        <inertia ixx="0" ixy="0" ixz="0" iyy="0" iyz="0" izz="0" />
-      </inertial>
       <visual>
         <geometry>
@@ -114,5 +106,5 @@
       <origin xyz="${j0_xyz}" rpy="${j0_rpy}" />
       <axis xyz="1 0 0" />
-      <limit effort="16.0" lower="${j0_lower}" upper="${j0_upper}" velocity="25.0" />
+      <limit effort="24.0" lower="${j0_lower}" upper="${j0_upper}" velocity="20.0" />
       <dynamics damping="0.1" friction="0.48" />
     </joint>
@@ -122,5 +114,5 @@
       <origin xyz="${j1_xyz}" rpy="${j1_rpy}" />
       <axis xyz="1 0 0" />
-      <limit effort="16.0" lower="${j1_lower}" upper="${j1_upper}" velocity="25.0" />
+      <limit effort="24.0" lower="${j1_lower}" upper="${j1_upper}" velocity="20.0" />
       <dynamics damping="0.1" friction="0.48" />
     </joint>
@@ -130,5 +122,5 @@
       <origin xyz="${j2_xyz}" rpy="${j2_rpy}" />
       <axis xyz="1 0 0" />
-      <limit effort="16.0" lower="${j2_lower}" upper="${j2_upper}" velocity="25.0" />
+      <limit effort="24.0" lower="${j2_lower}" upper="${j2_upper}" velocity="20.0" />
       <dynamics damping="0.1" friction="0.48" />
     </joint>

File: urdf/hb50/hb50.urdf (robot description, URDF)
Before this commit: robot hb50, 17 links, 16 joints
Links:
- link fl_foot: mass 0 -> None
- link fr_foot: mass 0 -> None
- link rl_foot: mass 0 -> None
- link rl_l1: mass 1.784 -> 1.785
- link rr_foot: mass 0 -> None
- link rr_l1: mass 1.784 -> 1.785
Joints:
- joint fl_j0: limit lower=-1.570796 upper=1.047198 effort=16.0 velocity=25.0 -> lower=-1.570796 upper=1.047198 effort=24.0 velocity=20.0
- joint fl_j1: limit lower=-1.570796 upper=1.570796 effort=16.0 velocity=25.0 -> lower=-1.570796 upper=1.570796 effort=24.0 velocity=20.0
- joint fl_j2: limit lower=0 upper=2.70526 effort=16.0 velocity=25.0 -> lower=0 upper=2.70526 effort=24.0 velocity=20.0
- joint fr_j0: limit lower=-1.047198 upper=1.570796 effort=16.0 velocity=25.0 -> lower=-1.047198 upper=1.570796 effort=24.0 velocity=20.0
- joint fr_j1: limit lower=-1.570796 upper=1.570796 effort=16.0 velocity=25.0 -> lower=-1.570796 upper=1.570796 effort=24.0 velocity=20.0
- joint fr_j2: limit lower=-2.70526 upper=0 effort=16.0 velocity=25.0 -> lower=-2.70526 upper=0 effort=24.0 velocity=20.0
- joint rl_j0: limit lower=-1.047198 upper=1.570796 effort=16.0 velocity=25.0 -> lower=-1.047198 upper=1.570796 effort=24.0 velocity=20.0
- joint rl_j1: limit lower=-3.141593 upper=1.570796 effort=16.0 velocity=25.0 -> lower=-3.141593 upper=1.570796 effort=24.0 velocity=20.0
- joint rl_j2: limit lower=0 upper=2.70526 effort=16.0 velocity=25.0 -> lower=0 upper=2.70526 effort=24.0 velocity=20.0
- joint rr_j0: limit lower=-1.570796 upper=1.047198 effort=16.0 velocity=25.0 -> lower=-1.570796 upper=1.047198 effort=24.0 velocity=20.0
- joint rr_j1: limit lower=-1.570796 upper=3.141593 effort=16.0 velocity=25.0 -> lower=-1.570796 upper=3.141593 effort=24.0 velocity=20.0
- joint rr_j2: limit lower=-2.70526 upper=0 effort=16.0 velocity=25.0 -> lower=-2.70526 upper=0 effort=24.0 velocity=20.0

File: urdf/hb50/hb50.urdf.xacro (robot description, xacro)
@@ -3,4 +3,7 @@
   <!-- sim: none | mock | gazebo -->
   <xacro:arg name="sim" default="none" />
+  <xacro:if value="${'$(arg sim)' not in ['none', 'mock', 'gazebo']}">
+    ${xacro.fatal("sim must be none, mock or gazebo, got '$(arg sim)'")}
+  </xacro:if>
   <xacro:include filename="../common/_materials.xacro" />
   <xacro:include filename="_hb50_leg_macro.xacro" />
@@ -22,5 +25,4 @@
         <box size="0.196 0.152 0.124" />
       </geometry>
-      <material name="invisible" />
     </collision>
     <collision>
@@ -29,5 +31,4 @@
         <cylinder length="0.282" radius="0.056" />
       </geometry>
-      <material name="invisible" />
     </collision>
     <collision>
@@ -36,5 +37,4 @@
         <cylinder length="0.282" radius="0.056" />
       </geometry>
-      <material name="invisible" />
     </collision>
     <collision>
@@ -43,5 +43,4 @@
         <box size="0.048 0.128 0.048" />
       </geometry>
-      <material name="invisible" />
     </collision>
   </link>
@@ -53,5 +52,5 @@
     l0_inertial_xyz="0.021234 0.02611 -0.00004" l0_visual_rpy="3.141593 0 0"
     j1_xyz="0.06 0.0385 0" j1_rpy="0 0 -1.570796" j1_lower="-1.570796" j1_upper="1.570796"
-    l1_inertial_xyz="0.067316 -0.013171 0.002548" l1_ixx="0.006065" l1_iyy="0.003514" l1_izz="0.007592"
+    l1_mass="1.784" l1_inertial_xyz="0.067316 -0.013171 0.002548" l1_ixx="0.006065" l1_iyy="0.003514" l1_izz="0.007592"
     l1_visual_rpy="3.141593 0 0" l1_mesh="hb50_l1r.stl"
     l1_collision2_xyz="0.118 -0.134 0.013" l1_collision2_rpy="0.05 0 0"
@@ -69,5 +68,5 @@
     l0_inertial_xyz="0.021234 -0.02611 0.00004"
     j1_xyz="0.06 -0.0385 0" j1_rpy="0 0 1.570796" j1_lower="-1.570796" j1_upper="1.570796"
-    l1_inertial_xyz="0.067316 0.013171 0.002548" l1_ixx="0.006065" l1_iyy="0.003514" l1_izz="0.007592"
+    l1_mass="1.784" l1_inertial_xyz="0.067316 0.013171 0.002548" l1_ixx="0.006065" l1_iyy="0.003514" l1_izz="0.007592"
     l1_visual_rpy="0 3.141593 0" l1_mesh="hb50_l1l.stl"
     l1_collision2_xyz="0.118 0.134 0.013" l1_collision2_rpy="-0.05 0 0"
@@ -85,5 +84,5 @@
     l0_inertial_xyz="0.01945 0.024417 0" l0_visual_rpy="3.141593 0 0"
     j1_xyz="0.06 0.0385 0" j1_rpy="0 0 -1.570796" j1_lower="-3.141593" j1_upper="1.570796"
-    l1_inertial_xyz="0.067294 0.016208 0.002475" l1_ixx="0.005907" l1_iyy="0.003507" l1_izz="0.007445"
+    l1_mass="1.785" l1_inertial_xyz="0.067294 0.016208 0.002475" l1_ixx="0.005907" l1_iyy="0.003507" l1_izz="0.007445"
     l1_visual_rpy="0 3.141593 0" l1_mesh="hb50_l1l.stl"
     l1_collision2_xyz="0.118 0.134 0.013" l1_collision2_rpy="-0.05 0 0"
@@ -101,5 +100,5 @@
     l0_inertial_xyz="0.01945 -0.024417 0"
     j1_xyz="0.06 -0.0385 0" j1_rpy="0 0 1.570796" j1_lower="-1.570796" j1_upper="3.141593"
-    l1_inertial_xyz="0.067294 -0.016208 0.002475" l1_ixx="0.005907" l1_iyy="0.003507" l1_izz="0.007445"
+    l1_mass="1.785" l1_inertial_xyz="0.067294 -0.016208 0.002475" l1_ixx="0.005907" l1_iyy="0.003507" l1_izz="0.007445"
     l1_visual_rpy="3.141593 0 0" l1_mesh="hb50_l1r.stl"
     l1_collision2_xyz="0.118 -0.134 0.013" l1_collision2_rpy="0.05 0 0"

File: urdf/hb50w/_hb50w_leg_macro.xacro (robot description, xacro)
@@ -35,5 +35,4 @@
           <cylinder length="0.084" radius="0.051" />
         </geometry>
-        <material name="invisible" />
       </collision>
     </link>
@@ -57,5 +56,4 @@
           <cylinder length="0.11" radius="0.051" />
         </geometry>
-        <material name="invisible" />
       </collision>
       <collision>
@@ -64,5 +62,4 @@
           <box size="0.028 0.22 0.052" />
         </geometry>
-        <material name="invisible" />
       </collision>
     </link>
@@ -86,5 +83,4 @@
           <cylinder length="0.06" radius="0.012" />
         </geometry>
-        <material name="invisible" />
       </collision>
       <collision>
@@ -93,5 +89,4 @@
           <cylinder length="0.196" radius="0.016" />
         </geometry>
-        <material name="invisible" />
       </collision>
       <collision>
@@ -100,5 +95,4 @@
           <cylinder length="0.05" radius="0.028" />
         </geometry>
-        <material name="invisible" />
       </collision>
     </link>
@@ -121,5 +115,4 @@
           <cylinder length="0.024" radius="0.0679" />
         </geometry>
-        <material name="invisible" />
       </collision>
     </link>
@@ -130,5 +123,5 @@
       <origin xyz="${j0_xyz}" rpy="${j0_rpy}" />
       <axis xyz="1 0 0" />
-      <limit effort="16.0" lower="${j0_lower}" upper="${j0_upper}" velocity="25.0" />
+      <limit effort="24.0" lower="${j0_lower}" upper="${j0_upper}" velocity="20.0" />
       <dynamics damping="0.1" friction="0.48" />
     </joint>
@@ -138,5 +131,5 @@
       <origin xyz="${j1_xyz}" rpy="${j1_rpy}" />
       <axis xyz="1 0 0" />
-      <limit effort="16.0" lower="${j1_lower}" upper="${j1_upper}" velocity="25.0" />
+      <limit effort="24.0" lower="${j1_lower}" upper="${j1_upper}" velocity="20.0" />
       <dynamics damping="0.1" friction="0.48" />
     </joint>
@@ -146,5 +139,5 @@
       <origin xyz="${j2_xyz}" rpy="${j2_rpy}" />
       <axis xyz="1 0 0" />
-      <limit effort="16.0" lower="${j2_lower}" upper="${j2_upper}" velocity="25.0" />
+      <limit effort="24.0" lower="${j2_lower}" upper="${j2_upper}" velocity="20.0" />
       <dynamics damping="0.1" friction="0.48" />
     </joint>
@@ -154,6 +147,6 @@
       <origin xyz="${j3_xyz}" />
       <axis xyz="1 0 0" />
-      <limit effort="7.0" velocity="25.0" />
-      <dynamics damping="0.1" friction="0.48" />
+      <limit effort="7.0" velocity="40.0" />
+      <dynamics damping="0.1" friction="0.1" />
     </joint>
   </xacro:macro>

File: urdf/hb50w/hb50w.urdf (robot description, URDF)
Before this commit: robot hb50w, 17 links, 16 joints
Joints:
- joint fl_j0: limit lower=-1.570796 upper=1.047198 effort=16.0 velocity=25.0 -> lower=-1.570796 upper=1.047198 effort=24.0 velocity=20.0
- joint fl_j1: limit lower=-1.570796 upper=1.570796 effort=16.0 velocity=25.0 -> lower=-1.570796 upper=1.570796 effort=24.0 velocity=20.0
- joint fl_j2: limit lower=0 upper=2.70526 effort=16.0 velocity=25.0 -> lower=0 upper=2.70526 effort=24.0 velocity=20.0
- joint fl_j3: limit effort=7.0 velocity=25.0 -> effort=7.0 velocity=40.0
- joint fr_j0: limit lower=-1.047198 upper=1.570796 effort=16.0 velocity=25.0 -> lower=-1.047198 upper=1.570796 effort=24.0 velocity=20.0
- joint fr_j1: limit lower=-1.570796 upper=1.570796 effort=16.0 velocity=25.0 -> lower=-1.570796 upper=1.570796 effort=24.0 velocity=20.0
- joint fr_j2: limit lower=-2.70526 upper=0 effort=16.0 velocity=25.0 -> lower=-2.70526 upper=0 effort=24.0 velocity=20.0
- joint fr_j3: limit effort=7.0 velocity=25.0 -> effort=7.0 velocity=40.0
- joint rl_j0: limit lower=-1.047198 upper=1.570796 effort=16.0 velocity=25.0 -> lower=-1.047198 upper=1.570796 effort=24.0 velocity=20.0
- joint rl_j1: limit lower=-3.141593 upper=1.570796 effort=16.0 velocity=25.0 -> lower=-3.141593 upper=1.570796 effort=24.0 velocity=20.0
- joint rl_j2: limit lower=0 upper=2.70526 effort=16.0 velocity=25.0 -> lower=0 upper=2.70526 effort=24.0 velocity=20.0
- joint rl_j3: limit effort=7.0 velocity=25.0 -> effort=7.0 velocity=40.0
- joint rr_j0: limit lower=-1.570796 upper=1.047198 effort=16.0 velocity=25.0 -> lower=-1.570796 upper=1.047198 effort=24.0 velocity=20.0
- joint rr_j1: limit lower=-1.570796 upper=3.141593 effort=16.0 velocity=25.0 -> lower=-1.570796 upper=3.141593 effort=24.0 velocity=20.0
- joint rr_j2: limit lower=-2.70526 upper=0 effort=16.0 velocity=25.0 -> lower=-2.70526 upper=0 effort=24.0 velocity=20.0
- joint rr_j3: limit effort=7.0 velocity=25.0 -> effort=7.0 velocity=40.0

File: urdf/hb50w/hb50w.urdf.xacro (robot description, xacro)
@@ -3,4 +3,7 @@
   <!-- sim: none | mock | gazebo -->
   <xacro:arg name="sim" default="none" />
+  <xacro:if value="${'$(arg sim)' not in ['none', 'mock', 'gazebo']}">
+    ${xacro.fatal("sim must be none, mock or gazebo, got '$(arg sim)'")}
+  </xacro:if>
   <xacro:include filename="../common/_materials.xacro" />
   <xacro:include filename="_hb50w_leg_macro.xacro" />
@@ -22,5 +25,4 @@
         <box size="0.196 0.152 0.124" />
       </geometry>
-      <material name="invisible" />
     </collision>
     <collision>
@@ -29,5 +31,4 @@
         <cylinder length="0.33" radius="0.056" />
       </geometry>
-      <material name="invisible" />
     </collision>
     <collision>
@@ -36,5 +37,4 @@
         <cylinder length="0.33" radius="0.056" />
       </geometry>
-      <material name="invisible" />
     </collision>
     <collision>
@@ -43,5 +43,4 @@
         <box size="0.048 0.128 0.048" />
       </geometry>
-      <material name="invisible" />
     </collision>
   </link>
