Commit message: fix: update hb50 link masses

File: urdf/hb50/hb50.urdf (robot description, URDF)
Before this commit: robot hb50, 17 links, 16 joints
Links:
- link body: mass 6.698 -> 7.812
- link fl_l0: mass 0.092 -> 0.107
- link fl_l1: mass 1.784 -> 2.081
- link fr_l0: mass 0.092 -> 0.107
- link fr_l1: mass 1.784 -> 2.081
- link rl_l0: mass 0.083 -> 0.097
- link rl_l1: mass 1.785 -> 2.082
- link rr_l0: mass 0.083 -> 0.097
- link rr_l1: mass 1.785 -> 2.082

File: urdf/hb50/hb50.urdf.xacro (robot description, xacro)
@@ -11,5 +11,5 @@
   <link name="body">
     <inertial>
-      <mass value="6.698" />
+      <mass value="7.812" />
       <inertia ixx="0.034280" ixy="0" ixz="0" iyy="0.053850" iyz="0" izz="0.073590" />
     </inertial>
@@ -49,8 +49,8 @@
     prefix="fr"
     j0_xyz="0.1405 -0.064 0" j0_lower="-1.047198" j0_upper="1.570796"
-    l0_mesh="hb50_l0f.stl" l0_mass="0.092" l0_ixx="0.000066961" l0_iyy="0.000070869" l0_izz="0.000062385"
+    l0_mesh="hb50_l0f.stl" l0_mass="0.107" l0_ixx="0.000066961" l0_iyy="0.000070869" l0_izz="0.000062385"
     l0_inertial_xyz="0.021234 0.02611 -0.00004" l0_visual_rpy="3.141593 0 0"
     j1_xyz="0.06 0.0385 0" j1_rpy="0 0 -1.570796" j1_lower="-1.570796" j1_upper="1.570796"
-    l1_mass="1.784" l1_inertial_xyz="0.067316 -0.013171 0.002548" l1_ixx="0.006065" l1_iyy="0.003514" l1_izz="0.007592"
+    l1_mass="2.081" l1_inertial_xyz="0.067316 -0.013171 0.002548" l1_ixx="0.006065" l1_iyy="0.003514" l1_izz="0.007592"
     l1_visual_rpy="3.141593 0 0" l1_mesh="hb50_l1r.stl"
     l1_collision2_xyz="0.118 -0.134 0.013" l1_collision2_rpy="0.05 0 0"
@@ -65,8 +65,8 @@
     prefix="fl"
     j0_xyz="0.1405 0.064 0" j0_lower="-1.570796" j0_upper="1.047198"
-    l0_mesh="hb50_l0f.stl" l0_mass="0.092" l0_ixx="0.000066961" l0_iyy="0.000070869" l0_izz="0.000062385"
+    l0_mesh="hb50_l0f.stl" l0_mass="0.107" l0_ixx="0.000066961" l0_iyy="0.000070869" l0_izz="0.000062385"
     l0_inertial_xyz="0.021234 -0.02611 0.00004"
     j1_xyz="0.06 -0.0385 0" j1_rpy="0 0 1.570796" j1_lower="-1.570796" j1_upper="1.570796"
-    l1_mass="1.784" l1_inertial_xyz="0.067316 0.013171 0.002548" l1_ixx="0.006065" l1_iyy="0.003514" l1_izz="0.007592"
+    l1_mass="2.081" l1_inertial_xyz="0.067316 0.013171 0.002548" l1_ixx="0.006065" l1_iyy="0.003514" l1_izz="0.007592"
     l1_visual_rpy="0 3.141593 0" l1_mesh="hb50_l1l.stl"
     l1_collision2_xyz="0.118 0.134 0.013" l1_collision2_rpy="-0.05 0 0"
@@ -81,8 +81,8 @@
     prefix="rl"
     j0_xyz="-0.1405 0.064 0" j0_rpy="0 0 -3.141593" j0_lower="-1.047198" j0_upper="1.570796"
-    l0_mesh="hb50_l0r.stl" l0_mass="0.083" l0_ixx="0.000048192" l0_iyy="0.000050964" l0_izz="0.000058424"
+    l0_mesh="hb50_l0r.stl" l0_mass="0.097" l0_ixx="0.000048192" l0_iyy="0.000050964" l0_izz="0.000058424"
     l0_inertial_xyz="0.01945 0.024417 0" l0_visual_rpy="3.141593 0 0"
     j1_xyz="0.06 0.0385 0" j1_rpy="0 0 -1.570796" j1_lower="-3.141593" j1_upper="1.570796"
-    l1_mass="1.785" l1_inertial_xyz="0.067294 0.016208 0.002475" l1_ixx="0.005907" l1_iyy="0.003507" l1_izz="0.007445"
+    l1_mass="2.082" l1_inertial_xyz="0.067294 0.016208 0.002475" l1_ixx="0.005907" l1_iyy="0.003507" l1_izz="0.007445"
     l1_visual_rpy="0 3.141593 0" l1_mesh="hb50_l1l.stl"
     l1_collision2_xyz="0.118 0.134 0.013" l1_collision2_rpy="-0.05 0 0"
@@ -97,8 +97,8 @@
     prefix="rr"
     j0_xyz="-0.1405 -0.064 0" j0_rpy="0 0 -3.141593" j0_lower="-1.570796" j0_upper="1.047198"
-    l0_mesh="hb50_l0r.stl" l0_mass="0.083" l0_ixx="0.000048192" l0_iyy="0.000050964" l0_izz="0.000058424"
+    l0_mesh="hb50_l0r.stl" l0_mass="0.097" l0_ixx="0.000048192" l0_iyy="0.000050964" l0_izz="0.000058424"
     l0_inertial_xyz="0.01945 -0.024417 0"
     j1_xyz="0.06 -0.0385 0" j1_rpy="0 0 1.570796" j1_lower="-1.570796" j1_upper="3.141593"
-    l1_mass="1.785" l1_inertial_xyz="0.067294 -0.016208 0.002475" l1_ixx="0.005907" l1_iyy="0.003507" l1_izz="0.007445"
+    l1_mass="2.082" l1_inertial_xyz="0.067294 -0.016208 0.002475" l1_ixx="0.005907" l1_iyy="0.003507" l1_izz="0.007445"
     l1_visual_rpy="3.141593 0 0" l1_mesh="hb50_l1r.stl"
     l1_collision2_xyz="0.118 -0.134 0.013" l1_collision2_rpy="0.05 0 0"
